Commit message: inverse dynamics controller

File: src/yumi-description/urdf/Gazebo/gazebo.urdf.xacro (robot description, xacro)
@@ -1,8 +1,48 @@
 <?xml version="1.0"?>
 <robot name="yumi" xmlns:xacro="http://www.ros.org/wiki/xacro">
-  <gazebo>
-    <plugin name="gazebo_ros_controller" filename="libgazebo_ros_control.so">
-      <robotNamespace>/yumi</robotNamespace>
-    </plugin>
-  </gazebo>
+  <xacro:macro name="ros_control_joint" params="name max_effort">
+    <joint name="${name}">
+      <command_interface name="effort">
+        <param name="min">-${max_effort}</param>
+        <param name="max">${max_effort}</param>
+      </command_interface>
+      <state_interface name="position">
+        <param name="initial_value">0.0</param>
+      </state_interface>
+      <state_interface name="velocity" />
+      <state_interface name="effort" />
+    </joint>
+  </xacro:macro>
+  <xacro:macro name="yumi_ros_control" params="name max_effort controller_path namespace">
+    <ros2_control name="IgnitionSystem" type="system">
+      <hardware>
+        <plugin>ign_ros2_control/IgnitionSystem</plugin>
+      </hardware>
+      <xacro:ros_control_joint name="${name}_joint_1_r" max_effort="${max_effort}" />
+      <xacro:ros_control_joint name="${name}_joint_2_r" max_effort="${max_effort}" />
+      <xacro:ros_control_joint name="${name}_joint_3_r" max_effort="${max_effort}" />
+      <xacro:ros_control_joint name="${name}_joint_4_r" max_effort="${max_effort}" />
+      <xacro:ros_control_joint name="${name}_joint_5_r" max_effort="${max_effort}" />
+      <xacro:ros_control_joint name="${name}_joint_6_r" max_effort="${max_effort}" />
+      <xacro:ros_control_joint name="${name}_joint_7_r" max_effort="${max_effort}" />
+      <xacro:ros_control_joint name="${name}_joint_1_l" max_effort="${max_effort}" />
+      <xacro:ros_control_joint name="${name}_joint_2_l" max_effort="${max_effort}" />
+      <xacro:ros_control_joint name="${name}_joint_3_l" max_effort="${max_effort}" />
+      <xacro:ros_control_joint name="${name}_joint_4_l" max_effort="${max_effort}" />
+      <xacro:ros_control_joint name="${name}_joint_5_l" max_effort="${max_effort}" />
+      <xacro:ros_control_joint name="${name}_joint_6_l" max_effort="${max_effort}" />
+      <xacro:ros_control_joint name="${name}_joint_7_l" max_effort="${max_effort}" />
+    </ros2_control>
+    <gazebo>
+      <plugin filename="ign_ros2_control-system"
+        name="ign_ros2_control::IgnitionROS2ControlPlugin">
+        <robot_param>robot_description</robot_param>
+        <robot_param_node>robot_state_publisher</robot_param_node>
+        <parameters>${controller_path}</parameters>
+        <ros>
+          <namespace>${namespace}</namespace>
+        </ros>
+      </plugin>
+    </gazebo>
+  </xacro:macro>
 </robot>

File: src/yumi-description/urdf/Grippers/yumi_servo_gripper.gazebo.xacro (robot description, xacro)
@@ -2,12 +2,4 @@
 <robot name="yumi_servo_gripper" xmlns:xacro="http://www.ros.org/wiki/xacro">
   <xacro:macro name="yumi_servo_gripper_gazebo" params="name">
-  <!-- Plugin for the mimic o/c joint - AFAIK, that shouldn't be necessary any more starting with Gazebo 3.0 -->
-    <!-- <gazebo>
-      <plugin name="mimic_plugin" filename="libgazebo_mimic_plugin.so">
-       <joint>${name}_joint</joint>
-        <mimicJoint>${name}_joint_m</mimicJoint>
-        <multiplier>1.0</multiplier>
-      </plugin>
-    </gazebo>  -->
     <!-- body -->
     <gazebo reference="${name}_base">

File: src/yumi-description/urdf/Grippers/yumi_servo_gripper.xacro (robot description, xacro)
@@ -1,107 +1,100 @@
 <?xml version="1.0"?>
 <robot name="yumi" xmlns:xacro="http://www.ros.org/wiki/xacro">
-    <!-- Import all Gazebo-customization elements, including Gazebo colors -->
-    <xacro:include filename="$(find yumi-description)/urdf/Grippers/yumi_servo_gripper.gazebo.xacro" />
-    <!-- Import Transmissions -->
-    <xacro:include filename="$(find yumi-description)/urdf/Grippers/yumi_servo_gripper.transmission.xacro" />
-    <!-- some constants -->
-    <xacro:property name="joint_damping" value="0.5" />
-    <xacro:property name="gripper_joint_damping" value="1.0" />
-    <xacro:property name="max_gripper_effort" value="20"/>
-    <xacro:property name="max_gripper_velocity" value="2"/>
-  <xacro:macro name="yumi_servo_gripper" params="parent name hardware_interface *origin">
-    <!--joint between {parent} and base-->
+  <!-- Import all Gazebo-customization elements, including Gazebo colors -->
+  <xacro:include filename="$(find yumi-description)/urdf/Grippers/yumi_servo_gripper.gazebo.xacro" />
+  <!-- Import Transmissions -->
+  <!-- <xacro:include filename="$(find
+  yumi-description)/urdf/Grippers/yumi_servo_gripper.transmission.xacro" /> -->
+  <xacro:macro name="yumi_servo_gripper" params="parent name collision_enabled *origin">
+    <!--joint
+    between {parent} and base-->
     <joint name="${parent}_joint" type="fixed">
-      <xacro:insert_block name="origin"/>
-      <parent link="${parent}"/>
-      <child link="${name}_base"/>
+      <xacro:insert_block name="origin" />
+      <parent link="${parent}" />
+      <child link="${name}_base" />
     </joint>
     <link name="${name}_base">
       <inertial>
-        <origin xyz="0 0 0" rpy="0 0 0"/>
-        <mass value="0.2"/>
-        <inertia ixx="0.0001"  ixy="0"  ixz="0" iyy="0.0001" iyz="0" izz="0.0001" />
+        <origin xyz="0 0 0" rpy="0 0 0" />
+        <mass value="0.2" />
+        <inertia ixx="0.0001" ixy="0" ixz="0" iyy="0.0001" iyz="0" izz="0.0001" />
       </inertial>
       <visual>
-        <origin xyz="0 0 0" rpy="0 0 0"/>
+        <origin xyz="0 0 0" rpy="0 0 0" />
         <geometry>
-          <mesh filename="package://yumi-description/meshes/gripper/base.stl"/>
+          <mesh filename="package://yumi-description/meshes/gripper/base.stl" />
         </geometry>
-        <material name="Light_Grey"/>
+        <material name="Light_Grey" />
       </visual>
-      <collision>
-        <origin xyz="0 0 0" rpy="0 0 0"/>
-        <geometry>
-          <mesh filename="package://yumi-description/meshes/gripper/coarse/base.stl"/>
-        </geometry>
-        <material name="Light_Grey"/>
-      </collision>
+      <xacro:if value="${collision_enabled}">
+        <collision>
+          <origin xyz="0 0 0" rpy="0 0 0" />
+          <geometry>
+            <mesh filename="package://yumi-description/meshes/gripper/coarse/base.stl" />
+          </geometry>
+          <material name="Light_Grey" />
+        </collision>
+      </xacro:if>
     </link>
     <!-- joint between base and right finger -->
-    <joint name="${name}_joint" type="prismatic">
-      <parent link="${name}_base"/>
-      <child link="${name}_finger_r"/>
-      <origin xyz="0 -0.0065 0.0837" rpy="0 0 0"/>
-      <axis xyz="-1 0 0"/>
-      <limit lower="0" upper="0.025"
-             effort="${max_gripper_effort}" velocity="${max_gripper_velocity}" />
-      <dynamics damping="${gripper_joint_damping}"/>
+    <joint name="${name}_joint" type="fixed">
+      <parent link="${name}_base" />
+      <child link="${name}_finger_r" />
+      <origin xyz="0 -0.0065 0.0837" rpy="0 0 0" />
     </joint>
     <link name="${name}_finger_r">
       <inertial>
-        <origin xyz="0 0 0" rpy="0 0 0"/>
-        <mass value="0.01"/>
-        <inertia ixx="0.000001"  ixy="0"  ixz="0" iyy="0.000001" iyz="0" izz="0.000001" />
+        <origin xyz="0 0 0" rpy="0 0 0" />
+        <mass value="0.01" />
+        <inertia ixx="0.000001" ixy="0" ixz="0" iyy="0.000001" iyz="0" izz="0.000001" />
       </inertial>
       <visual>
-        <origin xyz="0 0 0" rpy="0 0 0"/>
+        <origin xyz="0 0 0" rpy="0 0 0" />
         <geometry>
-          <mesh filename="package://yumi-description/meshes/gripper/finger.stl"/>
+          <mesh filename="package://yumi-description/meshes/gripper/finger.stl" />
         </geometry>
-        <material name="Blue"/>
+        <material name="Blue" />
       </visual>
-      <collision>
-        <origin xyz="0 0 0" rpy="0 0 0"/>
-        <geometry>
-          <mesh filename="package://yumi-description/meshes/gripper/coarse/finger.stl"/>
-        </geometry>
-        <material name="Blue"/>
-      </collision>
+      <xacro:if value="${collision_enabled}">
+        <collision>
+          <origin xyz="0 0 0" rpy="0 0 0" />
+          <geometry>
+            <mesh filename="package://yumi-description/meshes/gripper/coarse/finger.stl" />
+          </geometry>
+          <material name="Blue" />
+        </collision>
+      </xacro:if>
     </link>
-   <!-- joint between base and left finger -->
-    <joint name="${name}_joint_m" type="prismatic">
-      <parent link="${name}_base"/>
-      <child link="${name}_finger_l"/>
-      <origin xyz="0 0.0065 0.0837" rpy="0 0 ${PI}"/>
-      <axis xyz="-1 0 0"/>
-      <limit lower="0" upper="0.025"
-             effort="${max_gripper_effort}" velocity="${max_gripper_velocity}" />
-      <dynamics damping="${gripper_joint_damping}"/>
-      <mimic joint="${name}_joint"/>
+    <!-- joint between base and left finger -->
+    <joint name="${name}_joint_m" type="fixed">
+      <parent link="${name}_base" />
+      <child link="${name}_finger_l" />
+      <origin xyz="0 0.0065 0.0837" rpy="0 0 ${PI}" />
     </joint>
     <link name="${name}_finger_l">
       <inertial>
-        <origin xyz="0 0 0" rpy="0 0 0"/>
-        <mass value="0.01"/>
-        <inertia ixx="0.000001"  ixy="0"  ixz="0" iyy="0.000001" iyz="0" izz="0.000001" />
+        <origin xyz="0 0 0" rpy="0 0 0" />
+        <mass value="0.01" />
+        <inertia ixx="0.000001" ixy="0" ixz="0" iyy="0.000001" iyz="0" izz="0.000001" />
       </inertial>
       <visual>
-        <origin xyz="0 0 0" rpy="0 0 0"/>
+        <origin xyz="0 0 0" rpy="0 0 0" />
         <geometry>
-          <mesh filename="package://yumi-description/meshes/gripper/finger.stl"/>
+          <mesh filename="package://yumi-description/meshes/gripper/finger.stl" />
         </geometry>
-        <material name="Blue"/>
+        <material name="Blue" />
       </visual>
-      <collision>
-        <origin xyz="0 0 0" rpy="0 0 0"/>
-        <geometry>
-          <mesh filename="package://yumi-description/meshes/gripper/coarse/finger.stl"/>
-        </geometry>
-        <material name="Blue"/>
-      </collision>
+      <xacro:if value="${collision_enabled}">
+        <collision>
+          <origin xyz="0 0 0" rpy="0 0 0" />
+          <geometry>
+            <mesh filename="package://yumi-description/meshes/gripper/coarse/finger.stl" />
+          </geometry>
+          <material name="Blue" />
+        </collision>
+      </xacro:if>
     </link>
-     <!--Extensions -->
+    <!--Extensions -->
     <xacro:yumi_servo_gripper_gazebo name="${name}" />
-    <xacro:yumi_servo_gripper_transmission name="${name}" hardware_interface="${hardware_interface}"/>
   </xacro:macro>
 </robot>

File: src/yumi-description/urdf/yumi.transmission.xacro (robot description, xacro)
@@ -5,9 +5,9 @@
       <type>transmission_interface/SimpleTransmission</type>
       <joint name="${name}_joint_1_r">
-	<hardwareInterface>${hardware_interface}</hardwareInterface>
+        <hardwareInterface>${hardware_interface}</hardwareInterface>
       </joint>
       <actuator name="${name}_motor_1_r">
-	<hardwareInterface>${hardware_interface}</hardwareInterface>
-	<mechanicalReduction>1</mechanicalReduction>
+        <hardwareInterface>${hardware_interface}</hardwareInterface>
+        <mechanicalReduction>1</mechanicalReduction>
       </actuator>
     </transmission>
@@ -15,9 +15,9 @@
       <type>transmission_interface/SimpleTransmission</type>
       <joint name="${name}_joint_2_r">
-	<hardwareInterface>${hardware_interface}</hardwareInterface>
+        <hardwareInterface>${hardware_interface}</hardwareInterface>
       </joint>
       <actuator name="${name}_motor_2_r">
-	<hardwareInterface>${hardware_interface}</hardwareInterface>
-	<mechanicalReduction>1</mechanicalReduction>
+        <hardwareInterface>${hardware_interface}</hardwareInterface>
+        <mechanicalReduction>1</mechanicalReduction>
       </actuator>
     </transmission>
@@ -25,9 +25,9 @@
       <type>transmission_interface/SimpleTransmission</type>
       <joint name="${name}_joint_3_r">
-	<hardwareInterface>${hardware_interface}</hardwareInterface>
+        <hardwareInterface>${hardware_interface}</hardwareInterface>
       </joint>
       <actuator name="${name}_motor_3_r">
-	<hardwareInterface>${hardware_interface}</hardwareInterface>
-	<mechanicalReduction>1</mechanicalReduction>
+        <hardwareInterface>${hardware_interface}</hardwareInterface>
+        <mechanicalReduction>1</mechanicalReduction>
       </actuator>
     </transmission>
@@ -35,9 +35,9 @@
       <type>transmission_interface/SimpleTransmission</type>
       <joint name="${name}_joint_4_r">
-	<hardwareInterface>${hardware_interface}</hardwareInterface>
+        <hardwareInterface>${hardware_interface}</hardwareInterface>
       </joint>
       <actuator name="${name}_motor_4_r">
-	<hardwareInterface>${hardware_interface}</hardwareInterface>
-	<mechanicalReduction>1</mechanicalReduction>
+        <hardwareInterface>${hardware_interface}</hardwareInterface>
+        <mechanicalReduction>1</mechanicalReduction>
       </actuator>
     </transmission>
@@ -45,9 +45,9 @@
       <type>transmission_interface/SimpleTransmission</type>
       <joint name="${name}_joint_5_r">
-	<hardwareInterface>${hardware_interface}</hardwareInterface>
+        <hardwareInterface>${hardware_interface}</hardwareInterface>
       </joint>
       <actuator name="${name}_motor_5_r">
-	<hardwareInterface>${hardware_interface}</hardwareInterface>
-	<mechanicalReduction>1</mechanicalReduction>
+        <hardwareInterface>${hardware_interface}</hardwareInterface>
+        <mechanicalReduction>1</mechanicalReduction>
       </actuator>
     </transmission>
@@ -55,9 +55,9 @@
       <type>transmission_interface/SimpleTransmission</type>
       <joint name="${name}_joint_6_r">
-	<hardwareInterface>${hardware_interface}</hardwareInterface>
+        <hardwareInterface>${hardware_interface}</hardwareInterface>
       </joint>
       <actuator name="${name}_motor_6_r">
-	<hardwareInterface>${hardware_interface}</hardwareInterface>
-	<mechanicalReduction>1</mechanicalReduction>
+        <hardwareInterface>${hardware_interface}</hardwareInterface>
+        <mechanicalReduction>1</mechanicalReduction>
       </actuator>
     </transmission>
@@ -65,9 +65,9 @@
       <type>transmission_interface/SimpleTransmission</type>
       <joint name="${name}_joint_7_r">
-	<hardwareInterface>${hardware_interface}</hardwareInterface>
+        <hardwareInterface>${hardware_interface}</hardwareInterface>
       </joint>
       <actuator name="${name}_motor_7_r">
-	<hardwareInterface>${hardware_interface}</hardwareInterface>
-	<mechanicalReduction>1</mechanicalReduction>
+        <hardwareInterface>${hardware_interface}</hardwareInterface>
+        <mechanicalReduction>1</mechanicalReduction>
       </actuator>
     </transmission>
@@ -75,9 +75,9 @@
       <type>transmission_interface/SimpleTransmission</type>
       <joint name="${name}_joint_1_l">
-	<hardwareInterface>${hardware_interface}</hardwareInterface>
+        <hardwareInterface>${hardware_interface}</hardwareInterface>
       </joint>
       <actuator name="${name}_motor_1_l">
-	<hardwareInterface>${hardware_interface}</hardwareInterface>
-	<mechanicalReduction>1</mechanicalReduction>
+        <hardwareInterface>${hardware_interface}</hardwareInterface>
+        <mechanicalReduction>1</mechanicalReduction>
       </actuator>
     </transmission>
@@ -85,9 +85,9 @@
       <type>transmission_interface/SimpleTransmission</type>
       <joint name="${name}_joint_2_l">
-	<hardwareInterface>${hardware_interface}</hardwareInterface>
+        <hardwareInterface>${hardware_interface}</hardwareInterface>
       </joint>
       <actuator name="${name}_motor_2_l">
-	<hardwareInterface>${hardware_interface}</hardwareInterface>
-	<mechanicalReduction>1</mechanicalReduction>
+        <hardwareInterface>${hardware_interface}</hardwareInterface>
+        <mechanicalReduction>1</mechanicalReduction>
       </actuator>
     </transmission>
@@ -95,9 +95,9 @@
       <type>transmission_interface/SimpleTransmission</type>
       <joint name="${name}_joint_3_l">
-	<hardwareInterface>${hardware_interface}</hardwareInterface>
+        <hardwareInterface>${hardware_interface}</hardwareInterface>
       </joint>
       <actuator name="${name}_motor_3_l">
-	<hardwareInterface>${hardware_interface}</hardwareInterface>
-	<mechanicalReduction>1</mechanicalReduction>
+        <hardwareInterface>${hardware_interface}</hardwareInterface>
+        <mechanicalReduction>1</mechanicalReduction>
       </actuator>
     </transmission>
@@ -105,9 +105,9 @@
       <type>transmission_interface/SimpleTransmission</type>
       <joint name="${name}_joint_4_l">
-	<hardwareInterface>${hardware_interface}</hardwareInterface>
+        <hardwareInterface>${hardware_interface}</hardwareInterface>
       </joint>
       <actuator name="${name}_motor_4_l">
-	<hardwareInterface>${hardware_interface}</hardwareInterface>
-	<mechanicalReduction>1</mechanicalReduction>
+        <hardwareInterface>${hardware_interface}</hardwareInterface>
+        <mechanicalReduction>1</mechanicalReduction>
       </actuator>
     </transmission>
@@ -115,9 +115,9 @@
       <type>transmission_interface/SimpleTransmission</type>
       <joint name="${name}_joint_5_l">
-	<hardwareInterface>${hardware_interface}</hardwareInterface>
+        <hardwareInterface>${hardware_interface}</hardwareInterface>
       </joint>
       <actuator name="${name}_motor_5_l">
-	<hardwareInterface>${hardware_interface}</hardwareInterface>
-	<mechanicalReduction>1</mechanicalReduction>
+        <hardwareInterface>${hardware_interface}</hardwareInterface>
+        <mechanicalReduction>1</mechanicalReduction>
       </actuator>
     </transmission>
@@ -125,9 +125,9 @@
       <type>transmission_interface/SimpleTransmission</type>
       <joint name="${name}_joint_6_l">
-	<hardwareInterface>${hardware_interface}</hardwareInterface>
+        <hardwareInterface>${hardware_interface}</hardwareInterface>
       </joint>
       <actuator name="${name}_motor_6_l">
-	<hardwareInterface>${hardware_interface}</hardwareInterface>
-	<mechanicalReduction>1</mechanicalReduction>
+        <hardwareInterface>${hardware_interface}</hardwareInterface>
+        <mechanicalReduction>1</mechanicalReduction>
       </actuator>
     </transmission>
@@ -135,9 +135,9 @@
       <type>transmission_interface/SimpleTransmission</type>
       <joint name="${name}_joint_7_l">
-	<hardwareInterface>${hardware_interface}</hardwareInterface>
+        <hardwareInterface>${hardware_interface}</hardwareInterface>
       </joint>
       <actuator name="${name}_motor_7_l">
-	<hardwareInterface>${hardware_interface}</hardwareInterface>
-	<mechanicalReduction>1</mechanicalReduction>
+        <hardwareInterface>${hardware_interface}</hardwareInterface>
+        <mechanicalReduction>1</mechanicalReduction>
       </actuator>
     </transmission>

File: src/yumi-description/urdf/yumi.urdf.xacro (robot description, xacro)
@@ -1,43 +1,43 @@
 <?xml version="1.0"?>
 <robot name="yumi" xmlns:xacro="http://www.ros.org/wiki/xacro">
-    <!-- Import Rviz colors -->
-    <xacro:include filename="$(find yumi-description)/urdf/Util/materials.xacro" />
-    <!-- Import utilities -->
-    <xacro:include filename="$(find yumi-description)/urdf/Util/utilities.xacro" />
-    <!--Import
-    the yumi macro -->
-    <xacro:include filename="$(find yumi-description)/urdf/yumi.xacro" />
-    <!--Import
-    the yumi servo gripper macro -->
-    <xacro:include filename="$(find yumi-description)/urdf/Grippers/yumi_servo_gripper.xacro" />
-    <!-- Import Gazebo plugins -->
-    <!-- <xacro:include filename="$(find yumi-description)/urdf/Gazebo/gazebo.urdf.xacro" /> -->
-    <xacro:property name="yumi_parent" value="world" />
-    <!--yumi-->
-    <xacro:yumi name="yumi" hardware_interface="hardware_interface/$(arg arms_interface)"
-        parent="${yumi_parent}">
-        <origin xyz="0 0 0.1" rpy="0 0 0" />
-    </xacro:yumi>
-    <!--right
-    gripper-->
-    <xacro:yumi_servo_gripper name="gripper_r"
-        hardware_interface="hardware_interface/$(arg grippers_interface)" parent="yumi_link_7_r">
-        <origin xyz="0 0 0.007" rpy="0 0 ${PI}" />
-    </xacro:yumi_servo_gripper>
-    <!--left
-    gripper-->
-    <xacro:yumi_servo_gripper name="gripper_l"
-        hardware_interface="hardware_interface/$(arg grippers_interface)" parent="yumi_link_7_l">
-        <origin xyz="0 0 0.007" rpy="0 0 ${PI}" />
-    </xacro:yumi_servo_gripper>
-    <link name="world" />
-    <joint name="world_joint" type="fixed">
-        <parent link="world" />
-        <child link="yumi_base_link" />
-        <origin xyz="0 0 0.1" rpy="0 0 0" />
-    </joint>
-    <gazebo>
-        <plugin filename="ignition-gazebo-joint-state-publisher-system"
-            name="ignition::gazebo::systems::JointStatePublisher" />
-    </gazebo>
+  <!-- Import Rviz colors -->
+  <xacro:include filename="$(find yumi-description)/urdf/Util/materials.xacro" />
+  <!-- Import utilities -->
+  <xacro:include filename="$(find yumi-description)/urdf/Util/utilities.xacro" />
+  <!--Import
+  the yumi macro -->
+  <xacro:include filename="$(find yumi-description)/urdf/yumi.xacro" />
+  <!--Import
+  the yumi servo gripper macro -->
+  <xacro:include filename="$(find yumi-description)/urdf/Grippers/yumi_servo_gripper.xacro" />
+  <xacro:property name="yumi_parent" value="world" />
+  <!--yumi-->
+  <xacro:yumi
+    name="$(arg body_name)"
+    hardware_interface="hardware_interface/$(arg arms_interface)"
+    controller_path="$(arg controller_path)"
+    parent="${yumi_parent}"
+    namespace="$(arg namespace)"
+    collision_enabled="$(arg collision_enabled)"
+    max_effort="$(arg max_effort)">
+    <origin xyz="0 0 0.1" rpy="0 0 0" />
+  </xacro:yumi>
+  <!--right
+  gripper -->
+  <xacro:yumi_servo_gripper name="gripper_r" parent="yumi_link_7_r"
+    collision_enabled="$(arg collision_enabled)">
+    <origin xyz="0 0 0.007" rpy="0 0 ${PI}" />
+  </xacro:yumi_servo_gripper>
+  <!--left
+  gripper -->
+  <xacro:yumi_servo_gripper name="gripper_l" parent="yumi_link_7_l"
+    collision_enabled="$(arg collision_enabled)">
+    <origin xyz="0 0 0.007" rpy="0 0 ${PI}" />
+  </xacro:yumi_servo_gripper>
+  <link name="world" />
+  <joint name="world_joint" type="fixed">
+    <parent link="world" />
+    <child link="yumi_base_link" />
+    <origin xyz="0 0 0.1" rpy="0 0 0" />
+  </joint>
 </robot>
