Commit message: inverse dynamics controller

File: src/yumi-description/urdf/yumi.xacro (robot description, xacro)
@@ -5,8 +5,10 @@
   <!-- Import Transmissions -->
   <xacro:include filename="$(find yumi-description)/urdf/yumi.transmission.xacro" />
+  <!-- Import Gazebo Ros2 Control -->
+  <xacro:include filename="$(find yumi-description)/urdf/Gazebo/gazebo.urdf.xacro" />
   <!-- some constants -->
-  <xacro:property name="joint_damping" value="0.5" />
-  <xacro:property name="max_effort" value="300" />
-  <xacro:macro name="yumi" params="parent name hardware_interface *origin">
+  <xacro:property name="joint_damping" value="0.0" />
+  <xacro:macro name="yumi"
+    params="parent name hardware_interface controller_path namespace collision_enabled max_effort *origin">
     <link name="yumi_base_link"></link>
     <joint name="${name}_base_link_to_body" type="fixed">
@@ -28,11 +30,13 @@
         <material name="Light_Grey" />
       </visual>
-      <collision>
-        <origin xyz="0 0 0" rpy="0 0 0" />
-        <geometry>
-          <mesh filename="package://yumi-description/meshes/coarse/body.stl" />
-        </geometry>
-        <material name="Light_Grey" />
-      </collision>
+      <xacro:if value="${collision_enabled}">
+        <collision>
+          <origin xyz="0 0 0" rpy="0 0 0" />
+          <geometry>
+            <mesh filename="package://yumi-description/meshes/coarse/body.stl" />
+          </geometry>
+          <material name="Light_Grey" />
+        </collision>
+      </xacro:if>
     </link>
     <!--/////////////////////////////////////
@@ -61,11 +65,13 @@
         <material name="Grey" />
       </visual>
-      <collision>
-        <origin xyz="0 0 0" rpy="0 0 0" />
-        <geometry>
-          <mesh filename="package://yumi-description/meshes/coarse/link_1.stl" />
-        </geometry>
-        <material name="Grey" />
-      </collision>
+      <xacro:if value="${collision_enabled}">
+        <collision>
+          <origin xyz="0 0 0" rpy="0 0 0" />
+          <geometry>
+            <mesh filename="package://yumi-description/meshes/coarse/link_1.stl" />
+          </geometry>
+          <material name="Grey" />
+        </collision>
+      </xacro:if>
     </link>
     <!-- joint between link_1_r and link_2_r -->
@@ -92,11 +98,13 @@
         <material name="Grey" />
       </visual>
-      <collision>
-        <origin xyz="0 0 0" rpy="0 0 0" />
-        <geometry>
-          <mesh filename="package://yumi-description/meshes/coarse/link_2.stl" />
-        </geometry>
-        <material name="Grey" />
-      </collision>
+      <xacro:if value="${collision_enabled}">
+        <collision>
+          <origin xyz="0 0 0" rpy="0 0 0" />
+          <geometry>
+            <mesh filename="package://yumi-description/meshes/coarse/link_2.stl" />
+          </geometry>
+          <material name="Grey" />
+        </collision>
+      </xacro:if>
     </link>
     <!-- joint between link_2_r and link_3_r -->
@@ -123,11 +131,13 @@
         <material name="Grey" />
       </visual>
-      <collision>
-        <origin xyz="0 0 0" rpy="0 0 0" />
-        <geometry>
-          <mesh filename="package://yumi-description/meshes/coarse/link_3.stl" />
-        </geometry>
-        <material name="Grey" />
-      </collision>
+      <xacro:if value="${collision_enabled}">
+        <collision>
+          <origin xyz="0 0 0" rpy="0 0 0" />
+          <geometry>
+            <mesh filename="package://yumi-description/meshes/coarse/link_3.stl" />
+          </geometry>
+          <material name="Grey" />
+        </collision>
+      </xacro:if>
     </link>
     <!-- joint between link_3_r and link_4_r -->
@@ -154,11 +164,13 @@
         <material name="Grey" />
       </visual>
-      <collision>
-        <origin xyz="0 0 0" rpy="0 0 0" />
-        <geometry>
-          <mesh filename="package://yumi-description/meshes/coarse/link_4.stl" />
-        </geometry>
-        <material name="Grey" />
-      </collision>
+      <xacro:if value="${collision_enabled}">
+        <collision>
+          <origin xyz="0 0 0" rpy="0 0 0" />
+          <geometry>
+            <mesh filename="package://yumi-description/meshes/coarse/link_4.stl" />
+          </geometry>
+          <material name="Grey" />
+        </collision>
+      </xacro:if>
     </link>
     <!-- joint between link_4_r and link_5_r -->
@@ -185,11 +197,13 @@
         <material name="Grey" />
       </visual>
-      <collision>
-        <origin xyz="0 0 0" rpy="0 0 0" />
-        <geometry>
-          <mesh filename="package://yumi-description/meshes/coarse/link_5.stl" />
-        </geometry>
-        <material name="Grey" />
-      </collision>
+      <xacro:if value="${collision_enabled}">
+        <collision>
+          <origin xyz="0 0 0" rpy="0 0 0" />
+          <geometry>
+            <mesh filename="package://yumi-description/meshes/coarse/link_5.stl" />
+          </geometry>
+          <material name="Grey" />
+        </collision>
+      </xacro:if>
     </link>
     <!-- joint between link_5_r and link_6_r -->
@@ -216,11 +230,13 @@
         <material name="Grey" />
       </visual>
-      <collision>
-        <origin xyz="0 0 0" rpy="0 0 0" />
-        <geometry>
-          <mesh filename="package://yumi-description/meshes/coarse/link_6.stl" />
-        </geometry>
-        <material name="Grey" />
-      </collision>
+      <xacro:if value="${collision_enabled}">
+        <collision>
+          <origin xyz="0 0 0" rpy="0 0 0" />
+          <geometry>
+            <mesh filename="package://yumi-description/meshes/coarse/link_6.stl" />
+          </geometry>
+          <material name="Grey" />
+        </collision>
+      </xacro:if>
     </link>
     <!-- joint between link_6_r and link_7_r -->
@@ -247,11 +263,13 @@
         <material name="Grey" />
       </visual>
-      <collision>
-        <origin xyz="0 0 0" rpy="0 0 0" />
-        <geometry>
-          <mesh filename="package://yumi-description/meshes/coarse/link_7.stl" />
-        </geometry>
-        <material name="Grey" />
-      </collision>
+      <xacro:if value="${collision_enabled}">
+        <collision>
+          <origin xyz="0 0 0" rpy="0 0 0" />
+          <geometry>
+            <mesh filename="package://yumi-description/meshes/coarse/link_7.stl" />
+          </geometry>
+          <material name="Grey" />
+        </collision>
+      </xacro:if>
     </link>
     <!--/////////////////////////////////////
@@ -280,11 +298,13 @@
         <material name="Grey" />
       </visual>
-      <collision>
-        <origin xyz="0 0 0" rpy="0 0 0" />
-        <geometry>
-          <mesh filename="package://yumi-description/meshes/coarse/link_1.stl" />
-        </geometry>
-        <material name="Grey" />
-      </collision>
+      <xacro:if value="${collision_enabled}">
+        <collision>
+          <origin xyz="0 0 0" rpy="0 0 0" />
+          <geometry>
+            <mesh filename="package://yumi-description/meshes/coarse/link_1.stl" />
+          </geometry>
+          <material name="Grey" />
+        </collision>
+      </xacro:if>
     </link>
     <!-- joint between link_1_l and link_2_l -->
@@ -311,11 +331,13 @@
         <material name="Grey" />
       </visual>
-      <collision>
-        <origin xyz="0 0 0" rpy="0 0 0" />
-        <geometry>
-          <mesh filename="package://yumi-description/meshes/coarse/link_2.stl" />
-        </geometry>
-        <material name="Grey" />
-      </collision>
+      <xacro:if value="${collision_enabled}">
+        <collision>
+          <origin xyz="0 0 0" rpy="0 0 0" />
+          <geometry>
+            <mesh filename="package://yumi-description/meshes/coarse/link_2.stl" />
+          </geometry>
+          <material name="Grey" />
+        </collision>
+      </xacro:if>
     </link>
     <!-- joint between link_2_l and link_3_l -->
@@ -342,11 +364,13 @@
         <material name="Grey" />
       </visual>
-      <collision>
-        <origin xyz="0 0 0" rpy="0 0 0" />
-        <geometry>
-          <mesh filename="package://yumi-description/meshes/coarse/link_3.stl" />
-        </geometry>
-        <material name="Grey" />
-      </collision>
+      <xacro:if value="${collision_enabled}">
+        <collision>
+          <origin xyz="0 0 0" rpy="0 0 0" />
+          <geometry>
+            <mesh filename="package://yumi-description/meshes/coarse/link_3.stl" />
+          </geometry>
+          <material name="Grey" />
+        </collision>
+      </xacro:if>
     </link>
     <!-- joint between link_3_l and link_4_l -->
@@ -373,11 +397,13 @@
         <material name="Grey" />
       </visual>
-      <collision>
-        <origin xyz="0 0 0" rpy="0 0 0" />
-        <geometry>
-          <mesh filename="package://yumi-description/meshes/coarse/link_4.stl" />
-        </geometry>
-        <material name="Grey" />
-      </collision>
+      <xacro:if value="${collision_enabled}">
+        <collision>
+          <origin xyz="0 0 0" rpy="0 0 0" />
+          <geometry>
+            <mesh filename="package://yumi-description/meshes/coarse/link_4.stl" />
+          </geometry>
+          <material name="Grey" />
+        </collision>
+      </xacro:if>
     </link>
     <!-- joint between link_4_l and link_5_l -->
@@ -404,11 +430,13 @@
         <material name="Grey" />
       </visual>
-      <collision>
-        <origin xyz="0 0 0" rpy="0 0 0" />
-        <geometry>
-          <mesh filename="package://yumi-description/meshes/coarse/link_5.stl" />
-        </geometry>
-        <material name="Grey" />
-      </collision>
+      <xacro:if value="${collision_enabled}">
+        <collision>
+          <origin xyz="0 0 0" rpy="0 0 0" />
+          <geometry>
+            <mesh filename="package://yumi-description/meshes/coarse/link_5.stl" />
+          </geometry>
+          <material name="Grey" />
+        </collision>
+      </xacro:if>
     </link>
     <!-- joint between link_5_l and link_6_l -->
@@ -435,11 +463,13 @@
         <material name="Grey" />
       </visual>
-      <collision>
-        <origin xyz="0 0 0" rpy="0 0 0" />
-        <geometry>
-          <mesh filename="package://yumi-description/meshes/coarse/link_6.stl" />
-        </geometry>
-        <material name="Grey" />
-      </collision>
+      <xacro:if value="${collision_enabled}">
+        <collision>
+          <origin xyz="0 0 0" rpy="0 0 0" />
+          <geometry>
+            <mesh filename="package://yumi-description/meshes/coarse/link_6.stl" />
+          </geometry>
+          <material name="Grey" />
+        </collision>
+      </xacro:if>
     </link>
     <!-- joint between link_6_l and link_7_l -->
@@ -466,15 +496,19 @@
         <material name="Grey" />
       </visual>
-      <collision>
-        <origin xyz="0 0 0" rpy="0 0 0" />
-        <geometry>
-          <mesh filename="package://yumi-description/meshes/coarse/link_7.stl" />
-        </geometry>
-        <material name="Grey" />
-      </collision>
+      <xacro:if value="${collision_enabled}">
+        <collision>
+          <origin xyz="0 0 0" rpy="0 0 0" />
+          <geometry>
+            <mesh filename="package://yumi-description/meshes/coarse/link_7.stl" />
+          </geometry>
+          <material name="Grey" />
+        </collision>
+      </xacro:if>
     </link>
     <!--Extensions -->
     <xacro:yumi_gazebo name="${name}" />
-    <xacro:yumi_transmission name="${name}" hardware_interface="${hardware_interface}" />
+    <!-- <xacro:yumi_transmission name="${name}" hardware_interface="${hardware_interface}" /> -->
+    <xacro:yumi_ros_control name="${name}" max_effort="${max_effort}"
+      controller_path="${controller_path}" namespace="${namespace}" />
   </xacro:macro>
 </robot>
